File: board/board.kicad_pcb (KiCad board)
At the start: 2 copper layers, 21 x 13 mm, 1 part

Commit message: initial
Parts:
- added C1: d.n.p, Capacitor_SMD:C_1206_3216Metric, F.Cu at (150.8, 97.6)
- added J1: 019_100BASE-T_with_CT, on_edge:on_edge_2x05_device, F.Cu at (140.0, 96.5)
- added J2: 004_BASE-T_CT, on_edge:on_edge_2x05_host, F.Cu at (161.0, 96.5)
- added J3: LPJ4265BDNL, b135:LPJ4265BDNL, F.Cu at (145.6, 115.4)
- moved LOGO1 5.95 mm to (150.8, 93.1)
Routing:
- net /magjack/TX+: track 0.00 -> 31.5 mm
- net /magjack/CT3: track 0.00 -> 26.6 mm
- net /magjack/CT: track 0.00 -> 26.6 mm, vias 0 -> 2
- net /magjack/TX-: track 0.00 -> 25.0 mm
- net /magjack/CT4: track 0.00 -> 23.0 mm
- net Net-(C1-Pad1): track 0.00 -> 20.0 mm
- net /magjack/CT1: track 0.00 -> 19.1 mm, vias 0 -> 1
- net Net-(J1-Pad10): track 0.00 -> 19.1 mm, vias 0 -> 2
- net Net-(J1-Pad9): track 0.00 -> 18.0 mm, vias 0 -> 2
- net /magjack/RX+: track 0.00 -> 16.6 mm
- net /magjack/CT2: track 0.00 -> 14.6 mm, vias 0 -> 1
- net /magjack/RX-: track 0.00 -> 9.98 mm
- net /magjack/SH: track 0.00 -> 3.09 mm
Other:
- board size 21 x 13 mm -> 21 x 29 mm
- board text added: "osf.004"
- board text added: "osf.019"
- board text added: "osf.b135.v1.0"
