File: board/magjack.kicad_sch (KiCad schematic)
At the start: 1 part

Commit message: initial
Parts:
- J3: renamed from J?; MPN (none) -> LPJ4265BDNL
Changed lines of the file:
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@@
   (symbol (lib_id "b135:LPJ4265BDNL") (at 161.29 105.41 0) (unit 1)
     (in_bom yes) (on_board yes) (fields_autoplaced)
-    (property "Reference" "J?" (id 0) (at 177.8 104.1399 0)
+    (property "Reference" "J3" (id 0) (at 177.8 104.1399 0)
       (effects (font (size 1.27 1.27)) (justify left))
     )
@@
       (effects (font (size 1.27 1.27)) hide)
     )
-    (property "Datasheet" "" (id 3) (at 157.48 127 0)
+    (property "Datasheet" "https://www.l-p.com/file/datasheet/lpj4265bdnl.pdf" (id 3) (at 157.48 127 0)
       (effects (font (size 1.27 1.27)) hide)
     )
+    (property "MPN" "LPJ4265BDNL" (id 4) (at 161.29 105.41 0)
+      (effects (font (size 1.27 1.27)) hide)
+    )
